File: hardware/4_displays/4_displays.kicad_pcb (KiCad board)
At the start: 2 copper layers, 48.3 x 35.6 mm, 22 parts, among them J1 Conn_01x08_Male, J2 Conn_01x08_Male, J3 Conn_01x02_Male, Q1 BC807, Q2 BC807, Q3 BC807, Q4 BC807, U1 LTC-4627JG

Commit message: Correção do esquemático
Parts:
- J1, J2: value Conn_01x08_Male -> Conn_01x07_Male; footprint Connector_PinHeader_2.54mm:PinHeader_1x08_P2.54mm_Vertical -> Connector_PinHeader_2.54mm:PinHeader_1x07_P2.54mm_Vertical
- moved J2 33.6 mm to (83.8, 58.4), turned to -90 degrees
- moved J1 33.5 mm to (68.6, 87.6), turned to 90 degrees
- moved Q2 2.54 mm to (80.0, 74.9)
- moved R1 2.54 mm to (80.0, 63.5)
- moved R14 1.27 mm to (77.5, 63.5)
Connections:
- J1 pad 1: Net-(J1-Pad1) -> D1
- J1 pad 2: unconnected-(J1-Pad2) -> D2
- J1 pad 3: Net-(J1-Pad3) -> Net-(R6-Pad1)
- J1 pad 4: Net-(J1-Pad4) -> Net-(R7-Pad1)
- J1 pad 5: Net-(J1-Pad5) -> D3
- J1 pad 6: Net-(J1-Pad6) -> Net-(R8-Pad1)
- J1 pad 7: Net-(J1-Pad7) -> D4
- J2 pad 1: D1 -> Net-(R9-Pad1)
- J2 pad 2: D2 -> Net-(R1-Pad1)
- J2 pad 3: Net-(J2-Pad3) -> Net-(R14-Pad1)
- J2 pad 4: unconnected-(J2-Pad4) -> Net-(R2-Pad1)
- J2 pad 5: Net-(J2-Pad5) -> Net-(R3-Pad2)
- J2 pad 6: D3 -> Net-(R4-Pad1)
- J2 pad 7: Net-(J2-Pad7) -> Net-(R5-Pad2)
- R1 pad 1: Net-(J1-Pad3) -> Net-(R1-Pad1)
- R1 pad 2: CL1-2 -> F
- R14 pad 1: Net-(J1-Pad4) -> Net-(R14-Pad1)
- R14 pad 2: F -> CL1-2
- R2 pad 1: Net-(J1-Pad5) -> Net-(R2-Pad1)
- R3 pad 2: Net-(J1-Pad6) -> Net-(R3-Pad2)
- R4 pad 1: Net-(J1-Pad7) -> Net-(R4-Pad1)
- R5 pad 2: Net-(J1-Pad8) -> Net-(R5-Pad2)
- R6 pad 1: Net-(J2-Pad3) -> Net-(R6-Pad1)
- R7 pad 1: Net-(J2-Pad5) -> Net-(R7-Pad1)
- R8 pad 1: Net-(J2-Pad7) -> Net-(R8-Pad1)
- R9 pad 1: Net-(J1-Pad1) -> Net-(R9-Pad1)
Routing:
- net +3V3: track 65.1 -> 73.1 mm
- net Net-(J1-Pad3): track 5.14 -> 0.00 mm
- net Net-(R9-Pad1): track 0.00 -> 4.94 mm
- net Net-(J1-Pad4): track 4.61 -> 0.00 mm
- net Net-(R7-Pad1): track 0.00 -> 4.61 mm
- net Net-(R8-Pad1): track 0.00 -> 4.61 mm
- net Net-(R6-Pad1): track 0.00 -> 4.61 mm
- net Net-(R4-Pad1): track 0.00 -> 4.61 mm
- net Net-(R5-Pad2): track 0.00 -> 4.61 mm
- net Net-(R3-Pad2): track 0.00 -> 4.61 mm
- net Net-(R2-Pad1): track 0.00 -> 4.61 mm
- net Net-(R14-Pad1): track 0.00 -> 4.61 mm
- net Net-(R1-Pad1): track 0.00 -> 4.61 mm
- net Net-(J1-Pad8): track 4.09 -> 0.00 mm
- net Net-(J1-Pad6): track 4.09 -> 0.00 mm
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